File: Schematics/IsolatedAnalogRead.sch (KiCad schematic (older format))
At the start: 30 parts, among them J1 220V AC 50Hz, J2 Fo, Q1 BC548B, U1 LM741, U2 NE555

Commit message: Schematics V1
Other:
- note added: "400V"
- note added: "All the resistor values are in ohms.\n1/4W if no power specified."
- note added: "L\n"
- note added: "N\n"
- note added: "WARNING: This device has direct mains electrical connection! \nRisk of electric shock and/or measurement equipment damage\nif not handled properly."
Changed lines of the file:
@@
 encoding utf-8
 Sheet 1 1
-Title "Optoisolated Analog Voltmeter"
+Title "Analog Voltmeter Optocoupler Driver"
 Date "2018-08-12"
 Rev "1.0"
@@
 Text Notes 2150 1950 0    50   ~ 0
 1W\n
-Text Notes 1800 2350 1    50   ~ 0
-1W\n
 Wire Notes Line
 	1300 3150 6400 3150
@@
 P 7600 1700
 F 0 "R6" V 7393 1700 50  0000 C CNN
-F 1 "1M" V 7484 1700 50  0000 C CNN
+F 1 "1M" V 7600 1700 50  0000 C CNN
 F 2 "" V 7530 1700 50  0001 C CNN
 F 3 "~" H 7600 1700 50  0001 C CNN
@@
 Text Notes 6900 4400 0    67   ~ 0
 To optocoupler drive\ninput\n
+Text Notes 750  7550 0    118  ~ 24
+WARNING: This device has direct mains electrical connection! \nRisk of electric shock and/or measurement equipment damage\nif not handled properly.
+Text Notes 7100 7000 0    118  ~ 0
+All the resistor values are in ohms.\n1/4W if no power specified.
+Text Notes 7550 1650 0    50   ~ 0
+1W\n
+Text Notes 7500 2300 0    50   ~ 0
+400V
+Text Notes 1750 2800 0    50   ~ 0
+L\n
+Text Notes 1750 2900 0    50   ~ 0
+N\n
 $EndSCHEMATC

Commit message: PCB v0
Parts:
- added JP1: Jumper, Resistor_THT:R_Axial_DIN0204_L3.6mm_D1.6mm_P5.08mm_Horizontal, symbol Device:Jumper
- added JP2: Jumper, Resistor_THT:R_Axial_DIN0204_L3.6mm_D1.6mm_P7.62mm_Horizontal, symbol Device:Jumper
- added TP1: GND, TestPoint:TestPoint_THTPad_D1.0mm_Drill0.5mm, symbol Connector:TestPoint
- added TP2: VCC, TestPoint:TestPoint_THTPad_D1.0mm_Drill0.5mm, symbol Connector:TestPoint
- added TP3: VEE, TestPoint:TestPoint_THTPad_D1.0mm_Drill0.5mm, symbol Connector:TestPoint
- added TP4: Fo, TestPoint:TestPoint_THTPad_D1.0mm_Drill0.5mm, symbol Connector:TestPoint
- added TP5: Vread, TestPoint:TestPoint_THTPad_D1.0mm_Drill0.5mm, symbol Connector:TestPoint
- C1, C8: footprint (none) -> Capacitor_THT:C_Rect_L24.0mm_W10.1mm_P22.50mm_MKT
- C2: footprint (none) -> Capacitor_THT:C_Disc_D3.0mm_W1.6mm_P2.50mm
- C3, C4: footprint (none) -> Capacitor_THT:CP_Radial_D5.0mm_P2.00mm
- C5, C6, C7, C9: footprint (none) -> Capacitor_THT:C_Disc_D3.8mm_W2.6mm_P2.50mm
- D1, D3, D4, D7: footprint (none) -> lib:D_DO-41_SOD81_P7.62mm_Horizontal_PinsReversed
- D2: value !N4007 -> 1N4007; footprint (none) -> lib:D_DO-41_SOD81_P7.62mm_Horizontal_PinsReversed
- D5, D6: footprint (none) -> Diode_THT:D_DO-41_SOD81_P7.62mm_Horizontal
- J1: footprint (none) -> Connector_Wire:SolderWirePad_1x02_P5.08mm_Drill1.5mm
- J2: footprint (none) -> Connector_Wire:SolderWirePad_1x02_P3.81mm_Drill1mm
- Q1: footprint (none) -> Package_TO_SOT_THT:TO-92
- R1, R3, R4, R5, R7, R8, R9: footprint (none) -> Resistor_THT:R_Axial_DIN0207_L6.3mm_D2.5mm_P10.16mm_Horizontal
- R2, R6: footprint (none) -> Resistor_THT:R_Axial_Power_L25.0mm_W6.4mm_P27.94mm
- U1, U2: footprint (none) -> Package_DIP:DIP-8_W7.62mm_LongPads
Connections:
- wire segments 105 -> 125
